File: Baguette.kicad_pcb (KiCad board)
At the start: 2 copper layers, 25.1 x 35.6 mm, 6 parts, among them J1 Conn_01x03_Male, J2 Conn_01x03_Male, J3 Conn_01x01_Male, J4 Conn_01x01_Male, U1 ECC83

Commit message: Update to latest KiCAD version
Parts:
- removed REF**: foxlogo, logos:foxlogo
- J1, J2: footprint Pin_Headers:Pin_Header_Straight_1x03_Pitch2.54mm -> Connector_PinHeader_2.54mm:PinHeader_1x03_P2.54mm_Vertical
- J3, J4: footprint Pin_Headers:Pin_Header_Straight_1x01_Pitch2.54mm -> Connector_PinHeader_2.54mm:PinHeader_1x01_P2.54mm_Vertical
- U1: footprint Valves:VALVE-NOVAL_P -> Library:VALVE-NOVAL_P
Connections:
- U1 pad 9: Net-(U1-Pad9) -> unconnected-(U1C-F2-Pad9)
Other:
- net class Default removed
- net class Heater removed
- board text added: "${REVISION}"
- board text removed: "r02"

Commit message: Small updates
Parts:
- J1, J2: value Conn_01x03_Male -> Conn_01x03_Pin
- J3, J4: value Conn_01x01_Male -> Conn_01x01_Pin
- moved J2 14.5 mm to (139.7, 101.6)
- moved J3 14.5 mm to (139.7, 76.2)
- moved U1 14.5 mm to (141.0, 94.0)
- moved J1 14.5 mm to (127.0, 101.6)
- moved J4 14.5 mm to (127.0, 76.2)
Routing:
- net Net-(J2-Pin_3): track 25.2 -> 25.8 mm
- net Net-(J2-Pin_2): track 19.9 -> 20.4 mm
Other:
- outline, holes or cut-outs redrawn
- board text added: "Do Good ^-^"
- board text removed: "Do Good"
