File: Baguette.kicad_sch (KiCad schematic)
At the start: 5 parts, among them J1 Conn_01x03_Male, J2 Conn_01x03_Male, J3 Conn_01x01_Male, J4 Conn_01x01_Male, U1 ECC83

Commit message: Small updates
Parts:
- J1, J2: value Conn_01x03_Male -> Conn_01x03_Pin
- J3, J4: value Conn_01x01_Male -> Conn_01x01_Pin
Changed lines of the file:
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@@
     (stroke (width 0) (type default))
+  )
+  (netclass_flag "" (length 2.54) (shape round) (at 163.83 97.79 90) (fields_autoplaced)
+    (effects (font (size 1.27 1.27)) (justify left bottom))
+    (property "Netclass" "Heater" (at 161.29 97.1804 90)
+      (effects (font (size 1.27 1.27) italic) (justify left))
+    )
+  )
+  (netclass_flag "" (length 2.54) (shape round) (at 168.91 97.79 270) (fields_autoplaced)
+    (effects (font (size 1.27 1.27)) (justify right bottom))
+    (property "Netclass" "Heater" (at 171.45 97.1804 90)
+      (effects (font (size 1.27 1.27) italic) (justify left))
+    )
   )
   (symbol (lib_id "Valve:ECC83") (at 120.65 77.47 0) (unit 1)
@@
   )
   (symbol (lib_id "Connector:Conn_01x01_Pin") (at 163.83 104.14 90) (unit 1)
-    (in_bom yes) (on_board yes) (dnp no)
-    (property "Reference" "J3" (at 162.7124 100.2284 90)
+    (in_bom yes) (on_board yes) (dnp no) (fields_autoplaced)
+    (property "Reference" "J3" (at 162.56 102.235 90)
       (effects (font (size 1.27 1.27)) (justify left))
     )
-    (property "Value" "Conn_01x01_Male" (at 162.7124 102.5398 90)
+    (property "Value" "Conn_01x01_Pin" (at 162.56 104.775 90)
       (effects (font (size 1.27 1.27)) (justify left))
     )
@@
   )
   (symbol (lib_id "Connector:Conn_01x01_Pin") (at 168.91 104.14 90) (unit 1)
-    (in_bom yes) (on_board yes) (dnp no)
-    (property "Reference" "J4" (at 171.1452 100.2284 90)
+    (in_bom yes) (on_board yes) (dnp no) (fields_autoplaced)
+    (property "Reference" "J4" (at 170.18 102.235 90)
       (effects (font (size 1.27 1.27)) (justify right))
     )
-    (property "Value" "Conn_01x01_Male" (at 171.1452 102.5398 90)
+    (property "Value" "Conn_01x01_Pin" (at 170.18 104.775 90)
       (effects (font (size 1.27 1.27)) (justify right))
     )
@@
   )
   (symbol (lib_id "Connector:Conn_01x03_Pin") (at 99.06 104.14 0) (unit 1)
-    (in_bom yes) (on_board yes) (dnp no)
-    (property "Reference" "J2" (at 98.3488 103.5304 0)
-      (effects (font (size 1.27 1.27)) (justify right))
+    (in_bom yes) (on_board yes) (dnp no) (fields_autoplaced)
+    (property "Reference" "J2" (at 99.695 96.52 0)
+      (effects (font (size 1.27 1.27)))
     )
-    (property "Value" "Conn_01x03_Male" (at 98.3488 105.8418 0)
-      (effects (font (size 1.27 1.27)) (justify right))
+    (property "Value" "Conn_01x03_Pin" (at 99.695 99.06 0)
+      (effects (font (size 1.27 1.27)))
     )
     (property "Footprint" "Connector_PinHeader_2.54mm:PinHeader_1x03_P2.54mm_Vertical" (at 99.06 104.14 0)
@@
   )
   (symbol (lib_id "Connector:Conn_01x03_Pin") (at 99.06 77.47 0) (unit 1)
-    (in_bom yes) (on_board yes) (dnp no)
-    (property "Reference" "J1" (at 98.3488 76.8604 0)
-      (effects (font (size 1.27 1.27)) (justify right))
+    (in_bom yes) (on_board yes) (dnp no) (fields_autoplaced)
+    (property "Reference" "J1" (at 99.695 69.85 0)
+      (effects (font (size 1.27 1.27)))
     )
-    (property "Value" "Conn_01x03_Male" (at 98.3488 79.1718 0)
-      (effects (font (size 1.27 1.27)) (justify right))
+    (property "Value" "Conn_01x03_Pin" (at 99.695 72.39 0)
+      (effects (font (size 1.27 1.27)))
     )
     (property "Footprint" "Connector_PinHeader_2.54mm:PinHeader_1x03_P2.54mm_Vertical" (at 99.06 77.47 0)
